File: Tympan_AIC_Shield.kicad_pcb (KiCad board)
At the start: 4 copper layers, 38 x 40 mm, 49 parts, among them J1 SJ-3523-SMT-TR, J2 SJ-3524-SMT-TR-PI, P1 CONN_01X06, P2 CONN_01X06, P3 CONN_01X06, P4 CONN_01X06, P5 CONN_01X06, U2 TLV320AIC3206IRSBT, U3 74LVC1G66

Commit message: Cleaned silk. Need to breakout PDM connections
Parts:
- moved G*** 1.73 mm to (133.8, 79.5)
- moved G*** 1.63 mm to (133.8, 60.6)
Other:
- board text added: "Designed in Brooklyn, NY USA Made in Taipei, Taiwan"
- board text added: "TYMPAN AIC SHIELD"
- board text added: "Tympan AIC Shield"
- board text removed: "Designed in Brooklyn, NY"
- board text removed: "TYMPAN CODEC SHIELD"
- board text removed: "Tympan CODEC Shield"
Changed lines of the file:
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@@
   )
   (setup
-    (last_trace_width 0.2032)
+    (last_trace_width 0.25)
     (user_trace_width 0.1778)
     (user_trace_width 0.2032)
@@
   )
   (module Graphics:Tympan_LOGO (layer B.Cu)
-    (at 133.825 62.205 180)
+    (at 133.85 60.58 180)
     (attr smd)
     (fp_text reference G*** (at 0 0 180) (layer B.SilkS) hide
@@
   )
   (module Graphics:oshwa-logo-gear (layer B.Cu)
-    (at 133.85 77.755 180)
+    (at 133.85 79.48 180)
     (attr smd)
     (fp_text reference G*** (at 0 0 180) (layer B.SilkS) hide
@@
     )
   )
-  (gr_text "Tympan\nCODEC Shield" (at 124.85 84.28) (layer F.SilkS)
+  (gr_text "Tympan\nAIC Shield" (at 124.85 84.28) (layer F.SilkS)
     (effects (font (size 1 1) (thickness 0.2)) (justify left))
   )
@@
   (gr_arc (start 116.6 84.73) (end 114.85 84.73) (angle -90) (layer Edge.Cuts) (width 0.2))
   (gr_line (start 116.625 86.48) (end 151.075 86.48) (angle 90) (layer Edge.Cuts) (width 0.15))
-  (gr_text "www.tympan.org\ngithub.com/tympan" (at 133.85 69.78) (layer B.SilkS)
+  (gr_text "www.tympan.org\ngithub.com/tympan" (at 133.85 71.98) (layer B.SilkS)
     (effects (font (size 1 1) (thickness 0.2)) (justify mirror))
   )
-  (gr_text "Designed in Brooklyn, NY" (at 133.775 51.805) (layer B.SilkS)
+  (gr_text "Designed in Brooklyn, NY USA\nMade in Taipei, Taiwan" (at 133.75 52.98) (layer B.SilkS)
     (effects (font (size 1 1) (thickness 0.2)) (justify mirror))
   )
@@
   (gr_line (start 151.075 46.48) (end 116.625 46.48) (angle 90) (layer Edge.Cuts) (width 0.15))
   (gr_line (start 152.85 84.705) (end 152.85 48.255) (angle 90) (layer Edge.Cuts) (width 0.15))
-  (gr_text "TYMPAN CODEC SHIELD" (at 133.85 54.855) (layer B.SilkS)
+  (gr_text "TYMPAN AIC SHIELD" (at 133.85 68.48) (layer B.SilkS)
     (effects (font (size 1.524 1.524) (thickness 0.25)) (justify mirror))
   )

Commit message: added PDM breakout
Parts:
- added G***: LOGO, Graphics:Tympan_LOGO, F.Cu at (134.0, 53.6)
- added P6: CONN_01X06, Pin_Headers:Pin_Header_Straight_1x06_Pitch2.54mm, F.Cu at (145.8, 71.8)
- moved R13 3.35 mm to (133.7, 60.7)
- moved R14 3.35 mm to (133.7, 63.3)
- moved R17 3.35 mm to (133.7, 59.4)
- moved R12 3.35 mm to (133.7, 62.0)
- moved C5 0.69 mm to (138.9, 79.5)
- moved C4 0.58 mm to (137.0, 79.5)
- moved P2 0.05 mm to (148.4, 71.8)
Connections:
- net /RX_3 renamed /PDM_CLK
- net /TX_3 renamed /PDM_DAT
- net Net-(P1-Pad2) renamed /IN1_R
- net Net-(P1-Pad3) renamed /IN1_L
- net Net-(P1-Pad4) renamed /LOL
- net Net-(P1-Pad5) renamed /LOR
- U2 pad 12: Net-(U2-Pad12) -> /PDM_CLK1
- U2 pad 15: Net-(U2-Pad15) -> /PDM_DAT1
Routing:
- net /IN2_R_1: track 28.2 -> 43.2 mm, vias 3 -> 4
- net /PDM_CLK1: track 0.00 -> 14.5 mm, vias 0 -> 2
- net /PDM_DAT1: track 0.00 -> 14.3 mm, vias 0 -> 2
- net /IN2_L_1: track 20.2 -> 23.9 mm
- net /HPL: track 17.9 -> 14.5 mm
- net /HPR: track 21.2 -> 18.6 mm
- net Net-(J1-Pad3): track 26.0 -> 28.5 mm
- net /IN1_L_1: track 14.5 -> 16.9 mm
- net /IN1_R_1: track 16.7 -> 14.5 mm
- net GND: track 62.9 -> 60.9 mm, vias 13 -> 12
- net /M_BIAS_1: track 25.4 -> 23.5 mm
- net Net-(C12-Pad2): track 24.5 -> 22.8 mm
- net /DIN_1: track 20.6 -> 19.2 mm
- net Net-(J1-Pad2): track 7.21 -> 8.59 mm
- net /SS_2: track 0.67 -> 0.00 mm
